File: pcb/raspi_pico_christmas_tree/raspi_pico_christmas_tree.sch (KiCad schematic (older format))
At the start: 14 parts, among them J1 Barrel_Jack, J2 WS8212, J3 SSD1306, SW1 Button, U1 ESP8266-01_ESP-01, U2 SC0915, U3 24LC512

Commit message: add a bunch of pcb files mark pcb off todo list
Parts:
- C1: footprint (none) -> Capacitors_THT:C_Disc_D3.0mm_W2.0mm_P2.50mm
- D1: value LED_Dual_ACA -> LED_ACA; footprint (none) -> LEDs:LED_D5.0mm-3
- J1: value Barrel_Jack -> PWR; footprint (none) -> Connectors:BARREL_JACK
- J2: footprint (none) -> def-footprints:CONN_HEADER_1_3
- J3: footprint (none) -> Pin_Headers:Pin_Header_Straight_1x07_Pitch2.54mm
- R1, R2, R3, R4, R5: footprint (none) -> Resistors_THT:R_Axial_DIN0207_L6.3mm_D2.5mm_P10.16mm_Horizontal
- SW1: footprint (none) -> stomp:Switches-Push_switch_THD
- U1: value ESP8266-01_ESP-01 -> ESP-01; footprint XCVR_ESP8266-01/ESP-01 -> esp01:ESP-01
- U2: value SC0915 -> RaspiPico; footprint MODULE_SC0915 -> raspberrypi_pico:MODULE_SC0915
- U3: footprint (none) -> Housings_DIP:DIP-8_W7.62mm
Connections:
- net GND: now also U2.A (USB_SHIELD), U2.B (USB_SHIELD), U2.C (USB_SHIELD), U2.D (USB_SHIELD)
- no-connect marks 32 -> 31
Changed lines of the file:
@@
 EESchema Schematic File Version 4
+LIBS:raspi_pico_christmas_tree-cache
 EELAYER 29 0
 EELAYER END
@@
 Comment4 ""
 $EndDescr
-$Comp
-L Memory_EEPROM:24LC512 U3
-U 1 1 61AC357F
-P 5700 1400
-F 0 "U3" H 5900 1700 50  0000 C CNN
-F 1 "24LC512" H 5400 1700 50  0000 C CNN
-F 2 "" H 5700 1400 50  0001 C CNN
-F 3 "http://ww1.microchip.com/downloads/en/DeviceDoc/21754M.pdf" H 5700 1400 50  0001 C CNN
-	1    5700 1400
-	-1   0    0    -1
-$EndComp
-$Comp
-L Device:LED_Dual_ACA D1
-U 1 1 61AC681A
-P 3300 5500
-F 0 "D1" H 3300 5925 50  0000 C CNN
-F 1 "LED_Dual_ACA" H 3300 5834 50  0000 C CNN
-F 2 "" H 3300 5500 50  0001 C CNN
-F 3 "~" H 3300 5500 50  0001 C CNN
-	1    3300 5500
-	0    -1   -1   0
-$EndComp
-$Comp
-L Device:R R5
-U 1 1 61AC77CC
-P 6700 3500
-F 0 "R5" H 6770 3546 50  0000 L CNN
-F 1 "R" H 6770 3455 50  0000 L CNN
-F 2 "" V 6630 3500 50  0001 C CNN
-F 3 "~" H 6700 3500 50  0001 C CNN
-	1    6700 3500
-	1    0    0    -1
-$EndComp
-$Comp
-L Device:R R4
-U 1 1 61AC8223
-P 5050 1050
-F 0 "R4" H 5120 1096 50  0000 L CNN
-F 1 "R" H 5120 1005 50  0000 L CNN
-F 2 "" V 4980 1050 50  0001 C CNN
-F 3 "~" H 5050 1050 50  0001 C CNN
-	1    5050 1050
-	1    0    0    -1
-$EndComp
-$Comp
-L Device:R R1
-U 1 1 61AC8842
-P 3200 4900
-F 0 "R1" H 3270 4946 50  0000 L CNN
-F 1 "R" H 3270 4855 50  0000 L CNN
-F 2 "" V 3130 4900 50  0001 C CNN
-F 3 "~" H 3200 4900 50  0001 C CNN
-	1    3200 4900
-	-1   0    0    1
-$EndComp
-$Comp
-L Device:R R2
-U 1 1 61AC97E6
-P 3400 4900
-F 0 "R2" H 3470 4946 50  0000 L CNN
-F 1 "R" H 3470 4855 50  0000 L CNN
-F 2 "" V 3330 4900 50  0001 C CNN
-F 3 "~" H 3400 4900 50  0001 C CNN
-	1    3400 4900
-	1    0    0    -1
-$EndComp
-$Comp
-L Device:C C1
-U 1 1 61ACB887
-P 6700 3950
-F 0 "C1" H 6815 3996 50  0000 L CNN
-F 1 "C" H 6815 3905 50  0000 L CNN
-F 2 "" H 6738 3800 50  0001 C CNN
-F 3 "~" H 6700 3950 50  0001 C CNN
-	1    6700 3950
-	1    0    0    -1
-$EndComp
-$Comp
-L ESP8266-01_ESP-01:ESP8266-01_ESP-01 U1
-U 1 1 61ACC534
-P 2750 3850
-F 0 "U1" H 2750 4417 50  0000 C CNN
-F 1 "ESP8266-01_ESP-01" H 2750 4326 50  0000 C CNN
-F 2 "XCVR_ESP8266-01/ESP-01" H 2750 3850 50  0001 L BNN
-F 3 "" H 2750 3850 50  0001 L BNN
-F 4 "V1.2" H 2750 3850 50  0001 L BNN "PARTREV"
-F 5 "AI-Thinker" H 2750 3850 50  0001 L BNN "MANUFACTURER"
-F 6 "11.2 mm" H 2750 3850 50  0001 L BNN "MAXIMUM_PACKAGE_HEIGHT"
-F 7 "Manufacturer recommendations or IPC 7351B" H 2750 3850 50  0001 L BNN "STANDARD"
-	1    2750 3850
-	-1   0    0    -1
-$EndComp
-$Comp
-L raspberrypi_pico:SC0915 U2
-U 1 1 61ACE4E2
-P 5050 4350
-F 0 "U2" H 5050 6217 50  0000 C CNN
-F 1 "SC0915" H 5050 6126 50  0000 C CNN
-F 2 "MODULE_SC0915" H 5050 4350 50  0001 L BNN
-F 3 "" H 5050 4350 50  0001 L BNN
-F 4 "1.6" H 5050 4350 50  0001 L BNN "PARTREV"
-F 5 "Raspberry Pi" H 5050 4350 50  0001 L BNN "MANUFACTURER"
-F 6 "3.73mm" H 5050 4350 50  0001 L BNN "MAXIMUM_PACKAGE_HEIGHT"
-F 7 "Manufacturer Recommendations" H 5050 4350 50  0001 L BNN "STANDARD"
-	1    5050 4350
-	1    0    0    -1
-$EndComp
 Wire Wire Line
 	6050 2750 6250 2750
@@
 Wire Wire Line
 	3950 4750 4050 4750
-$Comp
-L Device:R R3
-U 1 1 61ACA97F
-P 4700 1050
-F 0 "R3" H 4770 1096 50  0000 L CNN
-F 1 "R" H 4770 1005 50  0000 L CNN
-F 2 "" V 4630 1050 50  0001 C CNN
-F 3 "~" H 4700 1050 50  0001 C CNN
-	1    4700 1050
-	1    0    0    -1
-$EndComp
 Wire Wire Line
 	3950 1300 4700 1300
@@
 Wire Wire Line
 	3200 4550 3200 4750
-$Comp
-L Switch:SW_Push_Dual SW1
-U 1 1 61AC50C9
-P 7350 3750
-F 0 "SW1" H 7350 4035 50  0000 C CNN
-F 1 "Button" H 7350 3944 50  0000 C CNN
-F 2 "" H 7350 3950 50  0001 C CNN
-F 3 "~" H 7350 3950 50  0001 C CNN
-	1    7350 3750
-	1    0    0    -1
-$EndComp
 NoConn ~ 7550 3950
 NoConn ~ 7150 3950
 NoConn ~ 2650 2200
-$Comp
-L Connector_Generic:Conn_01x03 J2
-U 1 1 61BD0D9B
-P 7250 4550
-F 0 "J2" H 7330 4592 50  0000 L CNN
-F 1 "WS8212" H 7330 4501 50  0000 L CNN
-F 2 "" H 7250 4550 50  0001 C CNN
-F 3 "~" H 7250 4550 50  0001 C CNN
-	1    7250 4550
-	1    0    0    -1
-$EndComp
 $Comp
 L power:GND #PWR014
@@
 Text Label 7650 4850 2    50   ~ 0
 GND
-$Comp
-L Connector_Generic:Conn_01x07 J3
-U 1 1 61BDC0E3
-P 7850 5150
-F 0 "J3" H 7930 5192 50  0000 L CNN
-F 1 "SSD1306" H 7930 5101 50  0000 L CNN
-F 2 "" H 7850 5150 50  0001 C CNN
-F 3 "~" H 7850 5150 50  0001 C CNN
-	1    7850 5150
-	1    0    0    -1
-$EndComp
 Wire Wire Line
 	6050 4050 6550 4050
@@
 NoConn ~ 4050 4350
 NoConn ~ 4050 4450
-$Comp
-L Connector:Barrel_Jack_Switch J1
-U 1 1 61C57C18
-P 2950 2200
-F 0 "J1" H 2720 2242 50  0000 R CNN
-F 1 "Barrel_Jack" H 3100 2400 50  0000 R CNN
-F 2 "" H 3000 2160 50  0001 C CNN
-F 3 "~" H 3000 2160 50  0001 C CNN
-	1    2950 2200
-	-1   0    0    -1
-$EndComp
 Wire Wire Line
 	3450 3950 4050 3950
@@
 Wire Wire Line
 	2500 2300 2400 2300
-NoConn ~ 6050 5650
+$Comp
+L power:GND #PWR0101
+U 1 1 61AE7882
+P 6150 5650
+F 0 "#PWR0101" H 6150 5400 50  0001 C CNN
+F 1 "GND" V 6150 5450 50  0000 C CNN
+F 2 "" H 6150 5650 50  0001 C CNN
+F 3 "" H 6150 5650 50  0001 C CNN
+	1    6150 5650
+	0    -1   -1   0
+$EndComp
+Wire Wire Line
+	6150 5650 6050 5650
+$Comp
+L Memory_EEPROM:24LC512 U3
+U 1 1 61AC357F
+P 5700 1400
+F 0 "U3" H 5900 1700 50  0000 C CNN
+F 1 "24LC512" H 5400 1700 50  0000 C CNN
+F 2 "Housings_DIP:DIP-8_W7.62mm" H 5700 1400 50  0001 C CNN
+F 3 "http://ww1.microchip.com/downloads/en/DeviceDoc/21754M.pdf" H 5700 1400 50  0001 C CNN
+	1    5700 1400
+	-1   0    0    -1
+$EndComp
+$Comp
+L Device:LED_Dual_ACA D1
+U 1 1 61AC681A
+P 3300 5500
+F 0 "D1" H 3300 5925 50  0000 C CNN
+F 1 "LED_ACA" H 3300 5834 50  0000 C CNN
+F 2 "LEDs:LED_D5.0mm-3" H 3300 5500 50  0001 C CNN
+F 3 "~" H 3300 5500 50  0001 C CNN
+	1    3300 5500
+	0    -1   -1   0
+$EndComp
+$Comp
+L Device:R R5
+U 1 1 61AC77CC
+P 6700 3500
+F 0 "R5" H 6770 3546 50  0000 L CNN
+F 1 "R" H 6770 3455 50  0000 L CNN
+F 2 "Resistors_THT:R_Axial_DIN0207_L6.3mm_D2.5mm_P10.16mm_Horizontal" V 6630 3500 50  0001 C CNN
+F 3 "~" H 6700 3500 50  0001 C CNN
+	1    6700 3500
+	1    0    0    -1
+$EndComp
+$Comp
+L Device:R R4
+U 1 1 61AC8223
+P 5050 1050
+F 0 "R4" H 5120 1096 50  0000 L CNN
+F 1 "R" H 5120 1005 50  0000 L CNN
+F 2 "Resistors_THT:R_Axial_DIN0207_L6.3mm_D2.5mm_P10.16mm_Horizontal" V 4980 1050 50  0001 C CNN
+F 3 "~" H 5050 1050 50  0001 C CNN
+	1    5050 1050
+	1    0    0    -1
+$EndComp
+$Comp
+L Device:R R1
+U 1 1 61AC8842
+P 3200 4900
+F 0 "R1" H 3270 4946 50  0000 L CNN
+F 1 "R" H 3270 4855 50  0000 L CNN
+F 2 "Resistors_THT:R_Axial_DIN0207_L6.3mm_D2.5mm_P10.16mm_Horizontal" V 3130 4900 50  0001 C CNN
+F 3 "~" H 3200 4900 50  0001 C CNN
+	1    3200 4900
+	-1   0    0    1
+$EndComp
+$Comp
+L Device:R R2
+U 1 1 61AC97E6
+P 3400 4900
+F 0 "R2" H 3470 4946 50  0000 L CNN
+F 1 "R" H 3470 4855 50  0000 L CNN
+F 2 "Resistors_THT:R_Axial_DIN0207_L6.3mm_D2.5mm_P10.16mm_Horizontal" V 3330 4900 50  0001 C CNN
+F 3 "~" H 3400 4900 50  0001 C CNN
+	1    3400 4900
+	1    0    0    -1
+$EndComp
+$Comp
+L Device:C C1
+U 1 1 61ACB887
+P 6700 3950
+F 0 "C1" H 6815 3996 50  0000 L CNN
+F 1 "C" H 6815 3905 50  0000 L CNN
+F 2 "Capacitors_THT:C_Disc_D3.0mm_W2.0mm_P2.50mm" H 6738 3800 50  0001 C CNN
+F 3 "~" H 6700 3950 50  0001 C CNN
+	1    6700 3950
+	1    0    0    -1
+$EndComp
+$Comp
+L ESP8266-01_ESP-01:ESP8266-01_ESP-01 U1
+U 1 1 61ACC534
+P 2750 3850
+F 0 "U1" H 2750 4417 50  0000 C CNN
+F 1 "ESP-01" H 2750 4326 50  0000 C CNN
+F 2 "esp01:ESP-01" H 2750 3850 50  0001 L BNN
+F 3 "" H 2750 3850 50  0001 L BNN
+F 4 "V1.2" H 2750 3850 50  0001 L BNN "PARTREV"
+F 5 "AI-Thinker" H 2750 3850 50  0001 L BNN "MANUFACTURER"
+F 6 "11.2 mm" H 2750 3850 50  0001 L BNN "MAXIMUM_PACKAGE_HEIGHT"
+F 7 "Manufacturer recommendations or IPC 7351B" H 2750 3850 50  0001 L BNN "STANDARD"
+	1    2750 3850
+	-1   0    0    -1
+$EndComp
+$Comp
+L Device:R R3
+U 1 1 61ACA97F
+P 4700 1050
+F 0 "R3" H 4770 1096 50  0000 L CNN
+F 1 "R" H 4770 1005 50  0000 L CNN
+F 2 "Resistors_THT:R_Axial_DIN0207_L6.3mm_D2.5mm_P10.16mm_Horizontal" V 4630 1050 50  0001 C CNN
+F 3 "~" H 4700 1050 50  0001 C CNN
+	1    4700 1050
+	1    0    0    -1
+$EndComp
+$Comp
+L Switch:SW_Push_Dual SW1
+U 1 1 61AC50C9
+P 7350 3750
+F 0 "SW1" H 7350 4035 50  0000 C CNN
+F 1 "Button" H 7350 3944 50  0000 C CNN
+F 2 "stomp:Switches-Push_switch_THD" H 7350 3950 50  0001 C CNN
+F 3 "~" H 7350 3950 50  0001 C CNN
+	1    7350 3750
+	1    0    0    -1
+$EndComp
+$Comp
+L Connector_Generic:Conn_01x03 J2
+U 1 1 61BD0D9B
+P 7250 4550
+F 0 "J2" H 7330 4592 50  0000 L CNN
+F 1 "WS8212" H 7330 4501 50  0000 L CNN
+F 2 "def-footprints:CONN_HEADER_1_3" H 7250 4550 50  0001 C CNN
+F 3 "~" H 7250 4550 50  0001 C CNN
+	1    7250 4550
+	1    0    0    -1
+$EndComp
+$Comp
+L Connector_Generic:Conn_01x07 J3
+U 1 1 61BDC0E3
+P 7850 5150
+F 0 "J3" H 7930 5192 50  0000 L CNN
+F 1 "SSD1306" H 7930 5101 50  0000 L CNN
+F 2 "Pin_Headers:Pin_Header_Straight_1x07_Pitch2.54mm" H 7850 5150 50  0001 C CNN
+F 3 "~" H 7850 5150 50  0001 C CNN
+	1    7850 5150
+	1    0    0    -1
+$EndComp
+$Comp
+L Connector:Barrel_Jack_Switch J1
+U 1 1 61C57C18
+P 2950 2200
+F 0 "J1" H 2720 2242 50  0000 R CNN
+F 1 "PWR" H 3100 2400 50  0000 R CNN
+F 2 "Connectors:BARREL_JACK" H 3000 2160 50  0001 C CNN
+F 3 "~" H 3000 2160 50  0001 C CNN
+	1    2950 2200
+	-1   0    0    -1
+$EndComp
+$Comp
+L raspberrypi_pico:SC0915 U2
+U 1 1 61ACE4E2
+P 5050 4350
+F 0 "U2" H 5050 6217 50  0000 C CNN
+F 1 "RaspiPico" H 5050 6126 50  0000 C CNN
+F 2 "raspberrypi_pico:MODULE_SC0915" H 5050 4350 50  0001 L BNN
+F 3 "" H 5050 4350 50  0001 L BNN
+F 4 "1.6" H 5050 4350 50  0001 L BNN "PARTREV"
+F 5 "Raspberry Pi" H 5050 4350 50  0001 L BNN "MANUFACTURER"
+F 6 "3.73mm" H 5050 4350 50  0001 L BNN "MAXIMUM_PACKAGE_HEIGHT"
+F 7 "Manufacturer Recommendations" H 5050 4350 50  0001 L BNN "STANDARD"
+	1    5050 4350
+	1    0    0    -1
+$EndComp
 $EndSCHEMATC
